File: hardware/kicad/bowen-nixie-device/bowen-nixie-device.kicad_pcb (KiCad board)
At the start: 2 copper layers, 29.2 x 29.2 mm, 119 parts, among them J1 Conn_01x02_Pin, J2 Conn_01x02_Pin, J3 Conn_01x04_Pin, Q1 SS8050, Q10 MMBTA42, Q11 MMBTA42, Q12 MMBTA42, Q13 MMBTA42, Q14 MMBTA42, Q15 MMBTA42, Q16 MMBTA42, Q17 MMBTA42, Q18 MMBTA42, Q19 MMBTA42, Q2 MPSA92, Q20 MMBTA42, Q21 MMBTA42, Q22 MMBTA42, Q23 MMBTA42, Q24 MMBTA42, Q25 MMBTA42, Q26 MMBTA42, Q27 MMBTA42, Q28 MMBTA42, Q29 MMBTA42, Q3 SS8050, Q30 MMBTA42, Q31 MMBTA42, Q32 MMBTA42, Q33 MMBTA42, Q34 MMBTA42, Q35 MMBTA42, Q36 MMBTA42, Q37 MMBTA42, Q38 MMBTA42, Q39 MMBTA42, Q4 MPSA92, Q40 MMBTA42, Q41 MMBTA42, Q42 MMBTA42, Q43 MMBTA42, Q44 MMBTA42, Q45 MMBTA42, Q46 MMBTA42, Q47 MMBTA42, Q48 MMBTA42, Q5 SS8050, Q6 MPSA92, Q7 SS8050, Q8 MPSA92, Q9 MMBTA42, U1 MOUDLE-SEEEDUINO-XIAO-ESP32C3, U11 NCH8200HV, U2 74HC595, U3 74HC595, U4 74HC595, U5 74HC595, U6 74HC595

Commit message: bowen progress
Parts:
- Q1, Q3, Q5, Q7: value SS8050 -> MMBTA42
- Q2, Q4, Q6, Q8: value MPSA92 -> MMBTA92; footprint Package_TO_SOT_THT:TO-92_Inline -> PCM_Package_TO_SOT_SMD_AKL:SOT-23
- moved U12 43.8 mm to (95.3, 94.2)
- moved R8 36.9 mm to (101.5, 60.2)
- moved Q7 36.7 mm to (67.6, 57.2), turned to 180 degrees
- moved R5 36.7 mm to (136.9, 60.2)
- moved R2 36.2 mm to (173.1, 60.2)
- moved Q1 36.1 mm to (175.2, 57.3), turned to 180 degrees
- moved R30 36.0 mm to (100.1, 75.2), turned to 90 degrees
- moved R40 36.0 mm to (136.1, 75.2), turned to 90 degrees
- moved R50 36.0 mm to (172.6, 75.2), turned to 90 degrees
- moved U2 35.9 mm to (165.1, 92.2)
- moved R31 35.6 mm to (100.1, 71.2), turned to 90 degrees
- moved R32 35.6 mm to (100.1, 67.2), turned to 90 degrees
- moved R41 35.6 mm to (136.1, 71.2), turned to 90 degrees
- moved Q6 35.6 mm to (97.1, 57.2), turned to 180 degrees
- moved R51 35.6 mm to (172.6, 71.2), turned to 90 degrees
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Connections:
- Q2 pad 1: 170V -> Net-(Q2-E)
- Q2 pad 2: Net-(Q2-B) -> 170V
- Q4 pad 1: 170V -> Net-(Q4-E)
- Q4 pad 2: Net-(Q4-B) -> 170V
- Q6 pad 1: 170V -> Net-(Q6-E)
- Q6 pad 2: Net-(Q6-B) -> 170V
- Q8 pad 1: 170V -> Net-(Q8-B)
- Q8 pad 2: Net-(Q8-B) -> 170V
- R2 pad 2: Net-(Q2-B) -> Net-(Q2-E)
- R3 pad 1: Net-(Q2-B) -> Net-(Q2-E)
- R5 pad 2: Net-(Q4-B) -> Net-(Q4-E)
- R6 pad 1: Net-(Q4-B) -> Net-(Q4-E)
- R8 pad 2: Net-(Q6-B) -> Net-(Q6-E)
- R9 pad 1: Net-(Q6-B) -> Net-(Q6-E)
Other:
- board size 29.2 x 29.2 mm -> 150 x 58.7 mm

Commit message: bowen layout progress
Parts:
- moved H3 24.0 mm to (53.2, 100.5)
- moved H1 2.01 mm to (53.2, 51.0)
- moved U1 1.12 mm to (77.1, 101.7)
- moved H2 0.75 mm to (196.8, 51.0)
- moved H4 0.37 mm to (196.8, 100.5)
- moved R9 0.17 mm to (100.6, 57.2)
Other:
- board size 150 x 58.7 mm -> 148.8 x 54.6 mm

Commit message: pcb tracing progress
Parts:
- removed U12: ~, Nixie:DS3231 Breakout
- moved Q1 1.10 mm to (176.3, 57.2)
- moved R10 0.65 mm to (68.2, 60.2)
- moved R11 0.51 mm to (64.6, 60.2)
- moved R3 0.45 mm to (172.6, 57.2)
- moved R7 0.40 mm to (104.7, 60.3)
- moved R6 0.33 mm to (136.6, 57.3)
- moved R8 0.33 mm to (101.1, 60.2)
- moved Q7 0.16 mm to (67.7, 57.3)
- moved Q3 0.16 mm to (140.3, 57.2)
- moved R5 0.15 mm to (137.1, 60.2)
- moved Q5 0.11 mm to (104.3, 57.2)
- moved R4 0.10 mm to (140.7, 60.3)
- moved R1 0.10 mm to (176.7, 60.3)
- moved R12 0.05 mm to (64.1, 57.3)
Routing:
- net 170V: track 0.00 -> 203.4 mm
- net SIN: track 0.00 -> 109.0 mm
- net SCLK: track 0.00 -> 104.7 mm
- net /T2IN6: track 0.00 -> 47.3 mm
- net /T1IN6: track 0.00 -> 44.5 mm
- net /T1IN8: track 0.00 -> 42.9 mm
- net /T4IN6: track 0.00 -> 41.8 mm
- net /T1IN9: track 0.00 -> 41.0 mm, vias 0 -> 2
- net /T3IN0: track 0.00 -> 40.4 mm, vias 0 -> 2
- net /T1IN5: track 0.00 -> 39.7 mm
- net /T4IN5: track 0.00 -> 37.3 mm
- net /T1IN4: track 0.00 -> 34.8 mm
- net /T3IN6: track 0.00 -> 34.1 mm
- net /T4IN4: track 0.00 -> 32.8 mm
- net /T3IN4: track 0.00 -> 32.6 mm
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- added copper zone on B.Cu, net GND
