File: hardware/kicad/bowen-nixie-device/bowen-nixie-device.kicad_pcb (KiCad board)
At the start: 2 copper layers, 148.8 x 54.6 mm, 118 parts, among them J1 Conn_01x02_Pin, J2 Conn_01x02_Pin, J3 Conn_01x04_Pin, Q1 MMBTA42, Q10 MMBTA42, Q11 MMBTA42, Q12 MMBTA42, Q13 MMBTA42, Q14 MMBTA42, Q15 MMBTA42, Q16 MMBTA42, Q17 MMBTA42, Q18 MMBTA42, Q19 MMBTA42, Q2 MMBTA92, Q20 MMBTA42, Q21 MMBTA42, Q22 MMBTA42, Q23 MMBTA42, Q24 MMBTA42, Q25 MMBTA42, Q26 MMBTA42, Q27 MMBTA42, Q28 MMBTA42, Q29 MMBTA42, Q3 MMBTA42, Q30 MMBTA42, Q31 MMBTA42, Q32 MMBTA42, Q33 MMBTA42, Q34 MMBTA42, Q35 MMBTA42, Q36 MMBTA42, Q37 MMBTA42, Q38 MMBTA42, Q39 MMBTA42, Q4 MMBTA92, Q40 MMBTA42, Q41 MMBTA42, Q42 MMBTA42, Q43 MMBTA42, Q44 MMBTA42, Q45 MMBTA42, Q46 MMBTA42, Q47 MMBTA42, Q48 MMBTA42, Q5 MMBTA42, Q6 MMBTA92, Q7 MMBTA42, Q8 MMBTA92, Q9 MMBTA42, U1 MOUDLE-SEEEDUINO-XIAO-ESP32C3, U11 NCH8200HV, U2 74HC595, U3 74HC595, U4 74HC595, U5 74HC595, U6 74HC595

Commit message: trace progress, gnd plane and most traces
Parts:
- moved J2 28.3 mm to (174.4, 101.3)
- moved J1 22.6 mm to (92.1, 101.5)
- moved J3 5.76 mm to (121.5, 101.3)
- moved Q7 1.00 mm to (68.7, 57.3)
- moved Q8 1.00 mm to (61.6, 57.2)
- moved R10 1.00 mm to (69.2, 60.2)
- moved R11 1.00 mm to (65.6, 60.2)
- moved R12 1.00 mm to (65.1, 57.3)
- moved Q44 0.55 mm to (189.1, 60.3)
- moved R48 0.55 mm to (185.6, 60.3)
- moved Q1 0.50 mm to (176.8, 57.2)
- moved Q2 0.50 mm to (169.6, 57.2)
- moved Q3 0.50 mm to (140.8, 57.2)
- moved Q4 0.50 mm to (133.6, 57.2)
- moved Q40 0.50 mm to (189.1, 76.2)
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Connections:
- U1 pad 1: AIN1 -> AIN4
- U1 pad 2: AIN2 -> AIN3
- U1 pad 3: AIN3 -> AIN2
- U1 pad 4: AIN4 -> AIN1
Routing:
- net +5V: track 0.00 -> 163.2 mm, vias 0 -> 11
- net ~OE: track 0.00 -> 110.7 mm, vias 0 -> 5
- net RCLK: track 19.0 -> 101.9 mm, vias 0 -> 4
- net /T4IN0: track 0.00 -> 54.1 mm, vias 0 -> 2
- net GND: track 0.95 -> 46.5 mm, vias 1 -> 50
- net /T1IN0: track 0.00 -> 38.2 mm, vias 0 -> 2
- net SOUT3: track 0.22 -> 15.6 mm
- net SOUT1: track 0.22 -> 15.6 mm
- net SOUT2: track 0.36 -> 15.5 mm
- net SOUT4: track 1.65 -> 15.3 mm
- net AOUT4: track 2.59 -> 0.00 mm
- net 170V: track 203.4 -> 200.9 mm
- net Net-(Q43-B): track 0.00 -> 2.44 mm
- net Net-(Q4-B): track 2.29 -> 4.62 mm
- net Net-(Q8-B): track 2.29 -> 4.62 mm
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
Commit message: layout final
Parts:
- U1: footprint Nixie:MOUDLE14P-SMD-2.54-21X17.8MM -> Nixie:XIAO-ESP32-C3-DIP
- moved U1 14.1 mm to (66.3, 92.6), turned to 180 degrees
Routing:
- net SIN: track 109.4 -> 107.8 mm
- net ~OE: track 110.7 -> 110.0 mm

Commit message: bowen passing drc layout
Parts:
- moved J2 7.39 mm to (167.0, 101.0)
- moved J1 0.52 mm to (92.1, 101.0)
- moved J3 0.31 mm to (121.5, 101.0)
Routing:
- net AIN1: track 0.00 -> 144.8 mm, vias 0 -> 2
- net AIN2: track 0.00 -> 112.0 mm, vias 0 -> 2
- net AIN3: track 0.00 -> 84.4 mm, vias 0 -> 2
- net SDA: track 0.00 -> 57.9 mm, vias 0 -> 1
- net SCL: track 0.00 -> 57.3 mm, vias 0 -> 1
- net AIN4: track 0.00 -> 46.5 mm, vias 0 -> 2
- net +5V: track 163.6 -> 159.5 mm
- net /T4IN0: track 54.1 -> 50.4 mm
- net AOUT4: track 0.00 -> 3.59 mm
- net ~OE: track 110.0 -> 112.4 mm, vias 5 -> 6
- net RCLK: track 102.0 -> 103.7 mm, vias 4 -> 5
- net SCLK: track 105.8 -> 107.5 mm, vias 0 -> 1
- net GND: track 46.2 -> 47.1 mm, vias 50 -> 49
- net /T4IN8: track 27.6 -> 28.2 mm

Commit message: bowen updates
Parts:
- added H5: MountingHole, MountingHole:MountingHole_2.2mm_M2_DIN965_Pad, F.Cu at (125.1, 81.9)
- added J4: Qwiic/Stemma QT, Connector_JST:JST_SH_BM04B-SRSS-TB_1x04-1MP_P1.00mm_Vertical, F.Cu at (173.1, 98.5)
- added J5: Conn_01x03_Pin, Connector_PinSocket_2.54mm:PinSocket_1x03_P2.54mm_Vertical, F.Cu at (53.1, 80.2)
- H1, H2, H3, H4: footprint MountingHole:MountingHole_2.2mm_M2 -> MountingHole:MountingHole_2.2mm_M2_DIN965_Pad
- R2: value 220k -> 470k
- moved J2 35.1 mm to (197.0, 82.8), turned to 0 degrees
Connections:
- U1 pad 10: unconnected-(U1-PA5_A9_D9_MISO-Pad10) -> EXT
Routing:
- net SDA: track 57.9 -> 108.1 mm
- net SCL: track 57.3 -> 104.5 mm
- net +5V: track 159.5 -> 185.3 mm, vias 11 -> 12
- net EXT: track 0.00 -> 17.0 mm
- net GND: track 47.1 -> 48.1 mm, vias 49 -> 50
Other:
- board text added: "Bowen Nixie Device"
- board text added: "C"
- board text added: "D"
- board text added: "G"
- board text added: "V"
