File: hardware/kicad/bowen-nixie-device/bowen-nixie-device.kicad_pcb (KiCad board)
At the start: 2 copper layers, 148.8 x 54.6 mm, 121 parts, among them J1 Conn_01x02_Pin, J2 Conn_01x02_Pin, J3 Conn_01x04_Pin, J4 Qwiic/Stemma QT, J5 Conn_01x03_Pin, Q1 MMBTA42, Q10 MMBTA42, Q11 MMBTA42, Q12 MMBTA42, Q13 MMBTA42, Q14 MMBTA42, Q15 MMBTA42, Q16 MMBTA42, Q17 MMBTA42, Q18 MMBTA42, Q19 MMBTA42, Q2 MMBTA92, Q20 MMBTA42, Q21 MMBTA42, Q22 MMBTA42, Q23 MMBTA42, Q24 MMBTA42, Q25 MMBTA42, Q26 MMBTA42, Q27 MMBTA42, Q28 MMBTA42, Q29 MMBTA42, Q3 MMBTA42, Q30 MMBTA42, Q31 MMBTA42, Q32 MMBTA42, Q33 MMBTA42, Q34 MMBTA42, Q35 MMBTA42, Q36 MMBTA42, Q37 MMBTA42, Q38 MMBTA42, Q39 MMBTA42, Q4 MMBTA92, Q40 MMBTA42, Q41 MMBTA42, Q42 MMBTA42, Q43 MMBTA42, Q44 MMBTA42, Q45 MMBTA42, Q46 MMBTA42, Q47 MMBTA42, Q48 MMBTA42, Q5 MMBTA42, Q6 MMBTA92, Q7 MMBTA42, Q8 MMBTA92, Q9 MMBTA42, U1 MOUDLE-SEEEDUINO-XIAO-ESP32C3, U11 NCH8200HV, U2 74HC595, U3 74HC595, U4 74HC595, U5 74HC595, U6 74HC595

Commit message: add bowen readme
Routing:
- net 170V: track 200.9 -> 198.6 mm

Commit message: bowen minor updates
Parts:
- J4: footprint Connector_JST:JST_SH_BM04B-SRSS-TB_1x04-1MP_P1.00mm_Vertical -> PCM_SparkFun-Connector:JST_1x04_P1.0mm_Vertical_SMD
- R11, R2, R5, R8: footprint Resistor_SMD:R_0603_1608Metric -> Resistor_SMD:R_1206_3216Metric
- R13, R14, R15, R16, R17, R18, R19, R20, R21, R22, R23, R24, R25, R26, R27, R28, R29, R30, R31, R32, R33, R34, R35, R36, R37, R38, R39, R40, R41, R42, R43, R44, R45, R46, R47, R48, R49, R50, R51, R52: value 4.7k -> 10k
- moved R11 6.78 mm to (70.8, 55.9)
- moved R8 6.78 mm to (106.8, 55.9)
- moved R2 6.70 mm to (178.7, 55.9)
- moved R5 6.70 mm to (142.7, 55.9)
- moved Q5 3.16 mm to (107.2, 59.3), turned to 0 degrees
- moved Q7 3.14 mm to (71.1, 59.3), turned to 0 degrees
- moved Q3 3.02 mm to (143.0, 59.3), turned to 0 degrees
- moved Q1 2.99 mm to (179.0, 59.3), turned to 0 degrees
- moved R4 2.25 mm to (139.2, 59.3), turned to 90 degrees
- moved R1 2.24 mm to (175.2, 59.3), turned to 90 degrees
- moved R10 2.17 mm to (67.2, 59.3), turned to 90 degrees
- moved R7 2.13 mm to (103.3, 59.3), turned to 90 degrees
- renumbered U6 to U2, U5 to U3, U3 to U5, U2 to U6
Connections:
- J3 pad 2: SDA -> SCL
- J3 pad 3: SCL -> SDA
- J4 pad 1: SCL -> GND
- J4 pad 2: SDA -> +5V
- J4 pad 3: +5V -> SDA
- J4 pad 4: GND -> SCL
Routing:
- net +5V: track 185.3 -> 182.3 mm, vias 12 -> 11
- net Net-(Q4-B): track 4.62 -> 7.39 mm
- net Net-(Q6-B): track 4.61 -> 7.11 mm
- net Net-(Q2-B): track 4.62 -> 7.09 mm
- net Net-(Q8-B): track 4.62 -> 7.01 mm
- net AIN1: track 144.8 -> 146.2 mm
- net SDA: track 108.1 -> 106.8 mm
- net AIN4: track 46.5 -> 47.8 mm
- net AIN3: track 84.4 -> 85.7 mm
- net SCLK: vias 1 -> 0

Commit message: final hardware updates maybe
Other:
- board text added: "WayWayWay"
Changed lines of the file:
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@@
 			)
 		)
-		(attr through_hole)
+		(attr through_hole exclude_from_bom dnp)
 		(duplicate_pad_numbers_are_jumpers no)
 		(fp_line
@@
 			)
 		)
+		(attr exclude_from_bom dnp)
 		(duplicate_pad_numbers_are_jumpers no)
 		(fp_circle
@@
 			)
 		)
-		(attr through_hole)
+		(attr through_hole exclude_from_bom dnp)
 		(duplicate_pad_numbers_are_jumpers no)
 		(fp_line
@@
 			)
 		)
+		(attr exclude_from_bom dnp)
 		(duplicate_pad_numbers_are_jumpers no)
 		(fp_circle
@@
 			)
 		)
-		(attr through_hole)
+		(attr through_hole exclude_from_bom dnp)
 		(duplicate_pad_numbers_are_jumpers no)
 		(fp_line
@@
 			(layers "F.Cu" "F.Mask" "F.Paste")
 			(roundrect_rratio 0.25)
-			(net "unconnected-(U6-QH'-Pad9)")
+			(net "unconnected-(U2-QH'-Pad9)")
 			(pinfunction "QH'_9")
 			(pintype "output+no_connect")
@@
 			)
 		)
+		(attr exclude_from_bom dnp)
 		(duplicate_pad_numbers_are_jumpers no)
 		(fp_circle
@@
 			)
 		)
+		(attr exclude_from_bom dnp)
 		(duplicate_pad_numbers_are_jumpers no)
 		(fp_circle
@@
 			)
 		)
-		(attr through_hole)
+		(attr through_hole exclude_from_bom dnp)
 		(duplicate_pad_numbers_are_jumpers no)
 		(fp_line
@@
 			)
 		)
-		(attr through_hole)
+		(attr through_hole exclude_from_bom dnp)
 		(duplicate_pad_numbers_are_jumpers no)
 		(fp_line
@@
 			)
 		)
-		(attr through_hole)
+		(attr through_hole exclude_from_bom dnp)
 		(duplicate_pad_numbers_are_jumpers no)
 		(fp_line
@@
 			)
 		)
-		(attr smd)
+		(attr smd exclude_from_bom dnp)
 		(duplicate_pad_numbers_are_jumpers no)
 		(fp_line
@@
 			)
 		)
-		(attr through_hole)
+		(attr through_hole exclude_from_bom dnp)
 		(duplicate_pad_numbers_are_jumpers no)
 		(fp_line
@@
 			)
 		)
-		(attr through_hole)
+		(attr through_hole exclude_from_bom dnp)
 		(duplicate_pad_numbers_are_jumpers no)
 		(fp_line
@@
 			)
 		)
-		(attr through_hole)
+		(attr through_hole exclude_from_bom dnp)
 		(duplicate_pad_numbers_are_jumpers no)
 		(fp_line
@@
 			)
 		)
+		(attr exclude_from_bom dnp)
 		(duplicate_pad_numbers_are_jumpers no)
 		(fp_circle
@@
 		)
 	)
+	(gr_text "WayWayWay"
+		(at 192.2 101 0)
+		(layer "B.SilkS")
+		(effects
+			(font
+				(size 1 1)
+				(thickness 0.15)
+			)
+			(justify left bottom mirror)
+		)
+	)
