File: hardware/kicad/IN7-180D-socket/IN7-180D-socket.kicad_pcb (KiCad board)
At the start: 2 copper layers, 31.8 x 31.8 mm, 5 parts, among them J1 Conn_01x08_Pin, J2 Conn_01x08_Pin, T1 IN-7

Commit message: final hardware updates maybe
Other:
- board text added: "WayWayWay"
- board text removed: "JLCJLCJLCJLC"
