File: hardware/kicad/IN7-270D-socket/IN7-270D-socket.kicad_pcb (KiCad board)
At the start: 2 copper layers, 31.8 x 31.8 mm, 5 parts, among them J1 Conn_01x08_Pin, J2 Conn_01x08_Pin, T1 IN-7

Commit message: final hardware updates maybe
Other:
- board text added: "WayWayWay"
- board text removed: "JLCJLCJLCJLC"
Changed lines of the file:
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@@
 		(at 50.8 50.8 90)
 		(property "Reference" "T1"
-			(at 0 -5.25 90)
+			(at 5.25 0 0)
 			(unlocked yes)
 			(layer "F.SilkS")
+			(hide yes)
 			(effects
 				(font
@@
 	)
 	(gr_text "270°"
-		(at 49.276 55.88 0)
+		(at 49.276 56 0)
 		(layer "F.SilkS")
 		(effects
@@
 		)
 	)
-	(gr_text "JLCJLCJLCJLC"
+	(gr_text "WayWayWay\n"
 		(at 55.88 66.04 0)
 		(layer "B.SilkS")
@@
 	)
 	(segment
-		(start 36.83 41.91)
-		(end 39.624 41.91)
-		(width 0.3)
-		(layer "B.Cu")
-		(net "Anode")
-	)
-	(segment
-		(start 44.069 37.465)
-		(end 46.99 37.465)
-		(width 0.3)
-		(layer "B.Cu")
-		(net "Anode")
-	)
-	(segment
-		(start 39.624 41.91)
-		(end 44.069 37.465)
-		(width 0.3)
-		(layer "B.Cu")
-		(net "Anode")
-	)
-	(segment
 		(start 62.23 57.15)
 		(end 64.77 59.69)
@@
 		(layer "F.Cu")
 		(net "K1")
+	)
+	(segment
+		(start 54.61 37.465)
+		(end 54.61 42.118225)
+		(width 0.3)
+		(layer "B.Cu")
+		(net "Net-(T1-Anode)")
+	)
+	(segment
+		(start 54.61 42.118225)
+		(end 54.243413 42.484812)
+		(width 0.3)
+		(layer "B.Cu")
+		(net "Net-(T1-Anode)")
 	)
 	(segment
@@
 	)
 	(segment
-		(start 54.61 37.465)
-		(end 54.61 42.118225)
-		(width 0.3)
-		(layer "B.Cu")
-		(net "Net-(T1-Anode)")
-	)
-	(segment
-		(start 54.61 42.118225)
-		(end 54.243413 42.484812)
-		(width 0.3)
-		(layer "B.Cu")
-		(net "Net-(T1-Anode)")
+		(start 36.83 41.91)
+		(end 39.624 41.91)
+		(width 0.3)
+		(layer "B.Cu")
+		(net "Anode")
+	)
+	(segment
+		(start 44.069 37.465)
+		(end 46.99 37.465)
+		(width 0.3)
+		(layer "B.Cu")
+		(net "Anode")
+	)
+	(segment
+		(start 39.624 41.91)
+		(end 44.069 37.465)
+		(width 0.3)
+		(layer "B.Cu")
+		(net "Anode")
 	)
 	(embedded_fonts no)
