File: hardware/kicad/IN4-0D-socket/IN4-0D-socket.kicad_pcb (KiCad board)
At the start: 2 copper layers, 31.8 x 31.8 mm, 5 parts, among them J1 Conn_01x08_Pin, J2 Conn_01x08_Pin, T1 IN-4

Commit message: final hardware updates maybe
Other:
- board text added: "WayWayWay"
- board text added: "e"
- board text removed: "JLCJLCJLCJLC"
Changed lines of the file:
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@@
 		)
 	)
-	(gr_text "JLCJLCJLCJLC"
+	(gr_text "e"
+		(at 51.18 56 0)
+		(layer "F.SilkS")
+		(effects
+			(font
+				(size 1 1)
+				(thickness 0.15)
+			)
+			(justify bottom)
+		)
+	)
+	(gr_text "WayWayWay"
 		(at 55.88 66.04 0)
 		(layer "B.SilkS")
@@
 	)
 	(segment
-		(start 41.275 37.465)
-		(end 36.83 41.91)
-		(width 0.3)
-		(layer "B.Cu")
-		(net "Anode")
-	)
-	(segment
-		(start 46.99 37.465)
-		(end 41.275 37.465)
-		(width 0.3)
-		(layer "B.Cu")
-		(net "Anode")
-	)
-	(segment
-		(start 50.803175 60.832915)
-		(end 63.627085 60.832915)
-		(width 0.3)
-		(layer "B.Cu")
-		(net "K1")
-	)
-	(segment
-		(start 49.703176 59.732916)
-		(end 50.803175 60.832915)
-		(width 0.3)
-		(layer "B.Cu")
-		(net "K1")
-	)
-	(segment
-		(start 63.627085 60.832915)
-		(end 64.77 59.69)
-		(width 0.3)
-		(layer "B.Cu")
-		(net "K1")
+		(start 55.884137 58.226457)
+		(end 58.633543 58.226457)
+		(width 0.3)
+		(layer "B.Cu")
+		(net "K4")
+	)
+	(segment
+		(start 60.78 56.08)
+		(end 60.78 53.6)
+		(width 0.3)
+		(layer "B.Cu")
+		(net "K4")
+	)
+	(segment
+		(start 60.78 53.6)
+		(end 64.77 49.61)
+		(width 0.3)
+		(layer "B.Cu")
+		(net "K4")
+	)
+	(segment
+		(start 58.633543 58.226457)
+		(end 60.78 56.08)
+		(width 0.3)
+		(layer "B.Cu")
+		(net "K4")
+	)
+	(segment
+		(start 58.514883 55.434655)
+		(end 61.37 52.579538)
+		(width 0.3)
+		(layer "F.Cu")
+		(net "K6")
+	)
+	(segment
+		(start 61.37 52.579538)
+		(end 61.37 45.31)
+		(width 0.3)
+		(layer "F.Cu")
+		(net "K6")
+	)
+	(segment
+		(start 61.37 45.31)
+		(end 64.77 41.91)
+		(width 0.3)
+		(layer "F.Cu")
+		(net "K6")
+	)
+	(segment
+		(start 43.84 58)
+		(end 47.88 53.96)
+		(width 0.3)
+		(layer "B.Cu")
+		(net "K8")
+	)
+	(segment
+		(start 36.83 57.15)
+		(end 37.68 58)
+		(width 0.3)
+		(layer "B.Cu")
+		(net "K8")
+	)
+	(segment
+		(start 47.88 53.96)
+		(end 57.575985 53.96)
+		(width 0.3)
+		(layer "B.Cu")
+		(net "K8")
+	)
+	(segment
+		(start 57.575985 53.96)
+		(end 59.739146 51.796839)
+		(width 0.3)
+		(layer "B.Cu")
+		(net "K8")
+	)
+	(segment
+		(start 37.68 58)
+		(end 43.84 58)
+		(width 0.3)
+		(layer "B.Cu")
+		(net "K8")
+	)
+	(segment
+		(start 54.61 37.465)
+		(end 54.61 39.19)
+		(width 0.3)
+		(layer "F.Cu")
+		(net "Net-(T1-Anode)")
+	)
+	(segment
+		(start 54.61 39.19)
+		(end 59.359593 43.939593)
+		(width 0.3)
+		(layer "F.Cu")
+		(net "Net-(T1-Anode)")
+	)
+	(segment
+		(start 59.359593 43.939593)
+		(end 59.359593 48.019222)
+		(width 0.3)
+		(layer "F.Cu")
+		(net "Net-(T1-Anode)")
+	)
+	(segment
+		(start 36.83 52.07)
+		(end 38.54 50.36)
+		(width 0.3)
+		(layer "B.Cu")
+		(net "K9")
+	)
+	(segment
+		(start 43.63 50.36)
+		(end 49.270586 44.719414)
+		(width 0.3)
+		(layer "B.Cu")
+		(net "K9")
+	)
+	(segment
+		(start 38.54 50.36)
+		(end 43.63 50.36)
+		(width 0.3)
+		(layer "B.Cu")
+		(net "K9")
+	)
+	(segment
+		(start 49.270586 44.719414)
+		(end 57.435293 44.719414)
+		(width 0.3)
+		(layer "B.Cu")
+		(net "K9")
+	)
+	(segment
+		(start 51.85 55.06)
+		(end 54.333968 52.576032)
+		(width 0.3)
+		(layer "F.Cu")
+		(net "K7")
+	)
+	(segment
+		(start 54.333968 52.576032)
+		(end 54.333968 42.522886)
+		(width 0.3)
+		(layer "F.Cu")
+		(net "K7")
+	)
+	(via
+		(at 51.85 55.06)
+		(size 0.6)
+		(drill 0.3)
+		(layers "F.Cu" "B.Cu")
+		(net "K7")
+	)
+	(segment
+		(start 37.68 60.54)
+		(end 36.83 59.69)
+		(width 0.3)
+		(layer "B.Cu")
+		(net "K7")
+	)
+	(segment
+		(start 51.85 55.06)
+		(end 46.37 60.54)
+		(width 0.3)
+		(layer "B.Cu")
+		(net "K7")
+	)
+	(segment
+		(start 46.37 60.54)
+		(end 37.68 60.54)
+		(width 0.3)
+		(layer "B.Cu")
+		(net "K7")
+	)
+	(segment
+		(start 46.832414 42.72176)
+		(end 43.63824 42.72176)
+		(width 0.3)
+		(layer "B.Cu")
+		(net "K10")
+	)
+	(segment
+		(start 43.63824 42.72176)
+		(end 36.83 49.53)
+		(width 0.3)
+		(layer "B.Cu")
+		(net "K10")
 	)
 	(segment
@@
 	)
 	(segment
-		(start 55.884137 58.226457)
-		(end 58.633543 58.226457)
-		(width 0.3)
-		(layer "B.Cu")
-		(net "K4")
-	)
-	(segment
-		(start 60.78 56.08)
-		(end 60.78 53.6)
-		(width 0.3)
-		(layer "B.Cu")
-		(net "K4")
-	)
-	(segment
-		(start 60.78 53.6)
-		(end 64.77 49.61)
-		(width 0.3)
-		(layer "B.Cu")
-		(net "K4")
-	)
-	(segment
-		(start 58.633543 58.226457)
-		(end 60.78 56.08)
-		(width 0.3)
-		(layer "B.Cu")
-		(net "K4")
-	)
-	(segment
 		(start 58.42 46.49)
 		(end 49.52 46.49)
@@
 	)
 	(segment
-		(start 58.514883 55.434655)
-		(end 61.37 52.579538)
-		(width 0.3)
-		(layer "F.Cu")
-		(net "K6")
-	)
-	(segment
-		(start 61.37 52.579538)
-		(end 61.37 45.31)
-		(width 0.3)
-		(layer "F.Cu")
-		(net "K6")
-	)
-	(segment
-		(start 61.37 45.31)
-		(end 64.77 41.91)
-		(width 0.3)
-		(layer "F.Cu")
-		(net "K6")
-	)
-	(segment
-		(start 51.85 55.06)
-		(end 54.333968 52.576032)
-		(width 0.3)
-		(layer "F.Cu")
-		(net "K7")
-	)
-	(segment
-		(start 54.333968 52.576032)
-		(end 54.333968 42.522886)
-		(width 0.3)
-		(layer "F.Cu")
-		(net "K7")
-	)
-	(via
-		(at 51.85 55.06)
-		(size 0.6)
-		(drill 0.3)
-		(layers "F.Cu" "B.Cu")
-		(net "K7")
-	)
-	(segment
-		(start 37.68 60.54)
-		(end 36.83 59.69)
-		(width 0.3)
-		(layer "B.Cu")
-		(net "K7")
-	)
-	(segment
-		(start 51.85 55.06)
-		(end 46.37 60.54)
-		(width 0.3)
-		(layer "B.Cu")
-		(net "K7")
-	)
-	(segment
-		(start 46.37 60.54)
-		(end 37.68 60.54)
-		(width 0.3)
-		(layer "B.Cu")
-		(net "K7")
-	)
-	(segment
-		(start 43.84 58)
-		(end 47.88 53.96)
-		(width 0.3)
-		(layer "B.Cu")
-		(net "K8")
-	)
-	(segment
-		(start 36.83 57.15)
-		(end 37.68 58)
-		(width 0.3)
-		(layer "B.Cu")
-		(net "K8")
-	)
-	(segment
-		(start 47.88 53.96)
-		(end 57.575985 53.96)
-		(width 0.3)
-		(layer "B.Cu")
-		(net "K8")
-	)
-	(segment
-		(start 57.575985 53.96)
-		(end 59.739146 51.796839)
-		(width 0.3)
-		(layer "B.Cu")
-		(net "K8")
-	)
-	(segment
-		(start 37.68 58)
-		(end 43.84 58)
-		(width 0.3)
-		(layer "B.Cu")
-		(net "K8")
-	)
-	(segment
-		(start 36.83 52.07)
-		(end 38.54 50.36)
-		(width 0.3)
-		(layer "B.Cu")
-		(net "K9")
-	)
-	(segment
-		(start 43.63 50.36)
-		(end 49.270586 44.719414)
-		(width 0.3)
-		(layer "B.Cu")
-		(net "K9")
-	)
-	(segment
-		(start 38.54 50.36)
-		(end 43.63 50.36)
-		(width 0.3)
-		(layer "B.Cu")
-		(net "K9")
-	)
-	(segment
-		(start 49.270586 44.719414)
-		(end 57.435293 44.719414)
-		(width 0.3)
-		(layer "B.Cu")
-		(net "K9")
-	)
-	(segment
-		(start 46.832414 42.72176)
-		(end 43.63824 42.72176)
-		(width 0.3)
-		(layer "B.Cu")
-		(net "K10")
-	)
-	(segment
-		(start 43.63824 42.72176)
-		(end 36.83 49.53)
-		(width 0.3)
-		(layer "B.Cu")
-		(net "K10")
-	)
-	(segment
-		(start 54.61 37.465)
-		(end 54.61 39.19)
-		(width 0.3)
-		(layer "F.Cu")
-		(net "Net-(T1-Anode)")
-	)
-	(segment
-		(start 54.61 39.19)
-		(end 59.359593 43.939593)
-		(width 0.3)
-		(layer "F.Cu")
-		(net "Net-(T1-Anode)")
-	)
-	(segment
-		(start 59.359593 43.939593)
-		(end 59.359593 48.019222)
-		(width 0.3)
-		(layer "F.Cu")
-		(net "Net-(T1-Anode)")
+		(start 50.803175 60.832915)
+		(end 63.627085 60.832915)
+		(width 0.3)
+		(layer "B.Cu")
+		(net "K1")
+	)
+	(segment
+		(start 49.703176 59.732916)
+		(end 50.803175 60.832915)
+		(width 0.3)
+		(layer "B.Cu")
+		(net "K1")
+	)
+	(segment
+		(start 63.627085 60.832915)
+		(end 64.77 59.69)
+		(width 0.3)
+		(layer "B.Cu")
+		(net "K1")
+	)
+	(segment
+		(start 41.275 37.465)
+		(end 36.83 41.91)
+		(width 0.3)
+		(layer "B.Cu")
+		(net "Anode")
+	)
+	(segment
+		(start 46.99 37.465)
+		(end 41.275 37.465)
+		(width 0.3)
+		(layer "B.Cu")
+		(net "Anode")
 	)
 	(embedded_fonts no)

Commit message: bowen fixes, final v1
Other:
- board text added: "0°"
- board text removed: "e"
Changed lines of the file:
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@@
 		)
 	)
-	(gr_text "e"
+	(gr_text "0°"
 		(at 51.18 56 0)
 		(layer "F.SilkS")
